Commit message: urdf com problemas no gazebo

File: description/baymax.urdf.xacro (robot description, xacro)
@@ -10,18 +10,121 @@
     <link name="world">
     </link>
-    <joint name="chassis_joint" type="fixed">
-        <origin xyz="-0.1 0.0 0.0" rpy="0.0 0.0 0.0"/>
+    <link name="body">
+        <xacro:inertial_body mass="18" length="0.8" radius="0.2">
+            <origin xyz="0.0 0.0 0.4" rpy="0.0 0.0 0.0"/>
+        </xacro:inertial_body>
+        <visual>
+            <geometry>
+                <cylinder radius="${body_radius}" length="${body_height}"/>
+            </geometry>
+        </visual>
+        <collision>
+            <geometry>
+                <cylinder radius="${body_radius}" length="${body_height}"/>
+            </geometry>
+        </collision>
+    </link>
+    <joint name="body_world_joint" type="fixed">
+        <origin xyz="0.0 0.0 ${body_height/2}" rpy="0.0 0.0 0.0"/>
         <parent link="world"/>
-        <child link="chassis"/>
-        <axis xyz="1 0.0 0.0"/>
+        <child link="body"/>
         <limit lower="0.0" upper="0.0" effort="0.0" velocity="0.0"/>
     </joint>
-    <link name="chassis">
+    <gazebo reference="body">
+        <material>Gazebo/White</material>
+    </gazebo>
+    <link name="left_wheel">
+        <xacro:inertial_body mass="0.1" length="0.03" radius="0.075">
+            <origin xyz="0.0 0.0 0.0" rpy="0.0 0.0 0.0"/>
+        </xacro:inertial_body>
         <visual>
-            <origin xyz="0.15 0 0.075" rpy="0.0 0.0 0.0"/>
             <geometry>
-                <box size="0.3 0.3 0.15"/>
+                <cylinder radius="${wheel_radius}" length="${wheel_thickness}"/>
             </geometry>
         </visual>
+        <collision>
+            <geometry>
+                <cylinder radius="${wheel_radius}" length="${wheel_thickness}"/>
+            </geometry>
+        </collision>
     </link>
+    <joint name="left_wheel_body_joint" type="continuous">
+        <origin xyz="-0.07 -0.215 -${body_height/2}" rpy="${pi/2} 0.0 0.0"/>
+        <parent link="body"/>
+        <child link="left_wheel"/>
+        <axis xyz="0.0 0.0 -1.0"/>
+        <limit lower="0.0" upper="0.0" effort="0.0" velocity="0.0"/>
+    </joint>
+    <gazebo reference="left_wheel">
+        <material>Gazebo/Red</material>
+    </gazebo>
+    <link name="right_wheel">
+        <xacro:inertial_body mass="0.1" length="0.03" radius="0.075">
+            <origin xyz="0.0 0.0 0.0" rpy="0.0 0.0 0.0"/>
+        </xacro:inertial_body>
+        <visual>
+            <geometry>
+                <cylinder radius="${wheel_radius}" length="${wheel_thickness}"/>
+            </geometry>
+        </visual>
+        <collision>
+            <geometry>
+                <cylinder radius="${wheel_radius}" length="${wheel_thickness}"/>
+            </geometry>
+        </collision>
+    </link>
+    <joint name="right_wheel_body_joint" type="continuous">
+        <origin xyz="-0.07 0.215 -${body_height/2}" rpy="-${pi/2} 0.0 0.0"/>
+        <parent link="body"/>
+        <child link="right_wheel"/>
+        <axis xyz="0.0 0.0 1.0"/>
+        <limit lower="0.0" upper="0.0" effort="0.0" velocity="0.0"/>
+    </joint>
+    <gazebo reference="right_wheel">
+        <material>Gazebo/Red</material>
+    </gazebo>
+    <link name="caster_wheel">
+        <xacro:inertial_body mass="0.1" length="0.03" radius="0.075">
+            <origin xyz="0.0 0.0 0.0" rpy="0.0 0.0 0.0"/>
+        </xacro:inertial_body>
+        <visual>
+            <geometry>
+                <cylinder radius="${wheel_radius/2}" length="${wheel_thickness}"/>
+            </geometry>
+        </visual>
+        <collision>
+            <geometry>
+                <cylinder radius="${wheel_radius/2}" length="${wheel_thickness}"/>
+            </geometry>
+        </collision>
+    </link>
+    <joint name="caster_wheel_body_joint" type="continuous">
+        <origin xyz="0.1 0.0 -${body_height/2 + wheel_radius/2}" rpy="-${pi/2} 0.0 0.0"/>
+        <parent link="body"/>
+        <child link="caster_wheel"/>
+        <axis xyz="0.0 0.0 1.0"/>
+        <limit lower="0.0" upper="0.0" effort="0.0" velocity="0.0"/>
+    </joint>
+    <link name="head">
+        <xacro:inertial_body mass="1" length="0.1" radius="0.1">
+            <origin xyz="0.0 0.0 0.0" rpy="0.0 0.0 0.0"/>
+        </xacro:inertial_body>
+        <visual>
+            <geometry>
+                <cylinder radius="${head_radius}" length="${head_height}"/>
+            </geometry>
+        </visual>
+        <collision>
+            <geometry>
+                <cylinder radius="${head_radius}" length="${head_height}"/>
+            </geometry>
+        </collision>
+    </link>
+    <joint name="head_body_joint" type="fixed">
+        <origin xyz="0.0 0.0 ${body_height/2 + head_height/2}" rpy="0.0 0.0 0.0"/>
+        <parent link="body"/>
+        <child link="head"/>
+        <axis xyz="0.0 0.0 0.0"/>
+        <limit lower="0.0" upper="0.0" effort="0.0" velocity="0.0"/>
+    </joint>
 </robot>

Commit message: baymax com teleop e lidar funcionando no gazebo

File: description/baymax.urdf.xacro (robot description, xacro)
@@ -2,4 +2,6 @@
 <robot xmlns:xacro="http://www.ros.org/wiki/xacro" name="baymax">
     <xacro:include filename="inertial_macros.urdf.xacro"/>
+    <xacro:include filename="gazebo_control.urdf.xacro"/>
+    <xacro:include filename="lidar.urdf.xacro"/>
     <xacro:property name="wheel_radius" value="0.075"/>
     <xacro:property name="body_height" value="0.8"/>
@@ -8,8 +10,8 @@
     <xacro:property name="head_radius" value="0.1"/>
     <xacro:property name="head_height" value="0.1"/>
-    <link name="world">
-    </link>
+    <!-- <link name="world">
+    </link> -->
     <link name="body">
-        <xacro:inertial_body mass="18" length="0.8" radius="0.2">
+        <xacro:inertial_body mass="1" length="0.8" radius="0.2">
             <origin xyz="0.0 0.0 0.4" rpy="0.0 0.0 0.0"/>
         </xacro:inertial_body>
@@ -25,10 +27,10 @@
         </collision>
     </link>
-    <joint name="body_world_joint" type="fixed">
-        <origin xyz="0.0 0.0 ${body_height/2}" rpy="0.0 0.0 0.0"/>
+    <!-- <joint name="body_world_joint" type="continuous">
+        <origin xyz="0.0 0.0 ${(body_height/2) + wheel_radius}" rpy="0.0 0.0 0.0"/>
         <parent link="world"/>
         <child link="body"/>
         <limit lower="0.0" upper="0.0" effort="0.0" velocity="0.0"/>
-    </joint>
+    </joint> -->
     <gazebo reference="body">
         <material>Gazebo/White</material>
@@ -57,5 +59,5 @@
     </joint>
     <gazebo reference="left_wheel">
-        <material>Gazebo/Red</material>
+        <material>Gazebo/Black</material>
     </gazebo>
     <link name="right_wheel">
@@ -82,8 +84,8 @@
     </joint>
     <gazebo reference="right_wheel">
-        <material>Gazebo/Red</material>
+        <material>Gazebo/Black</material>
     </gazebo>
     <link name="caster_wheel">
-        <xacro:inertial_body mass="0.1" length="0.03" radius="0.075">
+        <xacro:inertial_body mass="0.1" length="${wheel_thickness}" radius="${wheel_radius}">
             <origin xyz="0.0 0.0 0.0" rpy="0.0 0.0 0.0"/>
         </xacro:inertial_body>
@@ -99,4 +101,12 @@
         </collision>
     </link>
+    <!-- Tirar o atrito da roda boba -->
+    <gazebo reference="caster_wheel">
+        <material>
+            Gazebo/Black
+        </material>
+        <mu1 value="0.1"/>
+        <mu2 value="0.1"/>
+    </gazebo>
     <joint name="caster_wheel_body_joint" type="continuous">
         <origin xyz="0.1 0.0 -${body_height/2 + wheel_radius/2}" rpy="-${pi/2} 0.0 0.0"/>
@@ -107,5 +117,5 @@
     </joint>
     <link name="head">
-        <xacro:inertial_body mass="1" length="0.1" radius="0.1">
+        <xacro:inertial_body mass="0.05" length="0.1" radius="0.1">
             <origin xyz="0.0 0.0 0.0" rpy="0.0 0.0 0.0"/>
         </xacro:inertial_body>

File: description/inertial_macros.urdf.xacro (robot description, xacro)
@@ -5,5 +5,7 @@
             <xacro:insert_block name="origin"/>
             <mass value="${mass}"/>
-            <inertia ixx="1" ixy="1" ixz="1" iyy="1" iyz="1" izz="1"/>
+            <inertia    ixx="${(1/12) * mass * (3*radius*radius + length*length)}" ixy="0" ixz="0"
+                        iyy="${(1/12) * mass * (3*radius*radius + length*length)}" iyz="0"
+                        izz="${(1/2) * mass * (radius*radius)}"/>
         </inertial>
     </xacro:macro>

Commit message: urdf com lidar, camera e teleop via gamepad

File: description/baymax.urdf.xacro (robot description, xacro)
@@ -4,4 +4,5 @@
     <xacro:include filename="gazebo_control.urdf.xacro"/>
     <xacro:include filename="lidar.urdf.xacro"/>
+    <xacro:include filename="camera.urdf.xacro"/>
     <xacro:property name="wheel_radius" value="0.075"/>
     <xacro:property name="body_height" value="0.8"/>

File: description/camera.urdf.xacro (robot description, xacro)
@@ -1,3 +1,58 @@
-<?xml version="1.0"?>
-<robot xmlns:xacro="http://www.ros.org/wiki/xacro" name="robot_name">
+<?xml version="1.1" encoding="UTF-8"?>
+<robot xmlns:xacro="http://www.ros.org/wiki/xacro">
+    <joint name="camera_body_joint" type="fixed">
+        <parent link="body"/>
+        <child link="camera_link"/>
+        <origin xyz="0.18 0.0 0.42" rpy="0.0 0.0 0.0"/>
+    </joint>
+    <link name="camera_link">
+        <visual>
+            <geometry>
+                <box size="0.01 0.05 0.05"/>
+            </geometry>
+        </visual>
+        <collision>
+            <geometry>
+                <box size="0.1 0.1 0.1"/>
+            </geometry>
+        </collision>
+        <inertial>
+            <origin xyz="0.0 0.0 0.0" rpy="0.0 0.0 0.0"/>
+            <mass value="0.05"/>
+            <inertia ixx="1" ixy="0.0" ixz="0.0" iyy="1" iyz="0.0" izz="1"/>
+        </inertial>
+    </link>
+    <joint name="camera_optical_joint" type="fixed">
+        <origin xyz="0 0 0" rpy="${-pi/2} 0 ${-pi/2}" />
+        <parent link="camera_link" />
+        <child link="camera_link_optical" />
+    </joint>
+    <link name="camera_link_optical"></link>
+    <gazebo reference="camera_link">
+        <material>Gazebo/Red</material>
+        <sensor name="camera" type="camera">
+            <pose> 0 0 0 0 0 0 </pose>
+            <visualize>true</visualize>
+            <update_rate>10</update_rate>
+            <camera>
+                <camera>
+                    <horizontal_fov>1.089</horizontal_fov>
+                    <image>
+                        <format>R8G8B8</format>
+                        <width>640</width>
+                        <height>480</height>
+                    </image>
+                    <clip>
+                        <near>0.05</near>
+                        <far>8.0</far>
+                    </clip>
+                </camera>
+            </camera>
+            <plugin name="camera_controller" filename="libgazebo_ros_camera.so">
+                <plugin name="camera_controller" filename="libgazebo_ros_camera.so">
+                    <frame_name>camera_link_optical</frame_name>
+                </plugin>
+            </plugin>
+        </sensor>
+    </gazebo>
 </robot>

File: description/gazebo_control.urdf.xacro (robot description, xacro)
@@ -1,3 +1,3 @@
-<?xml version="1.0"?>
+<?xml version="1.1" encoding="UTF-8"?>
 <robot xmlns:xacro="http://www.ros.org/wiki/xacro">
     <gazebo>

File: description/inertial_macros.urdf.xacro (robot description, xacro)
@@ -1,3 +1,3 @@
-<?xml version="1.0"?>
+<?xml version="1.1" encoding="UTF-8"?>
 <robot xmlns:xacro="http://www.ros.org/wiki/xacro">
     <xacro:macro name="inertial_body" params="mass length radius *origin">

Commit message: ros2_control implementado

File: description/baymax.urdf.xacro (robot description, xacro)
@@ -2,11 +2,11 @@
 <robot xmlns:xacro="http://www.ros.org/wiki/xacro" name="baymax">
     <xacro:include filename="inertial_macros.urdf.xacro"/>
-    <xacro:include filename="gazebo_control.urdf.xacro"/>
+    <xacro:include filename="ros2_control.xacro"/>
     <xacro:include filename="lidar.urdf.xacro"/>
-    <xacro:include filename="camera.urdf.xacro"/>
+    <xacro:include filename="depth_camera.xacro"/>
     <xacro:property name="wheel_radius" value="0.075"/>
     <xacro:property name="body_height" value="0.8"/>
     <xacro:property name="body_radius" value="0.2"/>
-    <xacro:property name="wheel_thickness" value="0.03"/>
+    <xacro:property name="wheel_thickness" value="0.05"/>
     <xacro:property name="head_radius" value="0.1"/>
     <xacro:property name="head_height" value="0.1"/>
@@ -48,10 +48,10 @@
         <collision>
             <geometry>
-                <cylinder radius="${wheel_radius}" length="${wheel_thickness}"/>
+                <cylinder radius="${wheel_radius}" length="${wheel_thickness - 0.02}"/>
             </geometry>
         </collision>
     </link>
     <joint name="left_wheel_body_joint" type="continuous">
-        <origin xyz="-0.07 -0.215 -${body_height/2}" rpy="${pi/2} 0.0 0.0"/>
+        <origin xyz="-0.07 -0.22 -${body_height/2}" rpy="${pi/2} 0.0 0.0"/>
         <parent link="body"/>
         <child link="left_wheel"/>
@@ -78,5 +78,5 @@
     </link>
     <joint name="right_wheel_body_joint" type="continuous">
-        <origin xyz="-0.07 0.215 -${body_height/2}" rpy="-${pi/2} 0.0 0.0"/>
+        <origin xyz="-0.07 0.22 -${body_height/2}" rpy="-${pi/2} 0.0 0.0"/>
         <parent link="body"/>
         <child link="right_wheel"/>

Commit message: IMU implementado

File: description/baymax.urdf.xacro (robot description, xacro)
@@ -4,5 +4,8 @@
     <xacro:include filename="ros2_control.xacro"/>
     <xacro:include filename="lidar.urdf.xacro"/>
+    <!--Ainda n implementada completamente
     <xacro:include filename="depth_camera.xacro"/>
+    -->
+    <xacro:include filename="imu.urdf.xacro"/>
     <xacro:property name="wheel_radius" value="0.075"/>
     <xacro:property name="body_height" value="0.8"/>
@@ -28,5 +31,5 @@
         </collision>
     </link>
-    <!-- <joint name="body_world_joint" type="continuous">
+    <!-- <joint name="body_world_joint" type="fixed">
         <origin xyz="0.0 0.0 ${(body_height/2) + wheel_radius}" rpy="0.0 0.0 0.0"/>
         <parent link="world"/>

File: description/depth_camera.xacro (robot description, xacro)
@@ -4,5 +4,5 @@
         <parent link="body"/>
         <child link="camera_link"/>
-        <origin xyz="0.18 0.0 0.42" rpy="0.0 0.0 0.0"/>
+        <origin xyz="0.22 0 0.43" rpy="${pi/2} 0 0"/>
     </joint>
     <link name="camera_link">
@@ -24,5 +24,5 @@
     </link>
     <joint name="camera_optical_joint" type="fixed">
-        <origin xyz="0 0 0" rpy="${-pi/2} 0 ${-pi/2}" />
+        <origin xyz="0 0 0" rpy="${-pi/2} 0 ${-pi/2}"/>
         <parent link="camera_link" />
         <child link="camera_link_optical" />
@@ -31,5 +31,5 @@
     <gazebo reference="camera_link">
         <material>Gazebo/Red</material>
-        <sensor name="camera" type="camera">
+        <sensor name="camera" type="depth">
             <pose> 0 0 0 0 0 0 </pose>
             <visualize>true</visualize>
@@ -38,5 +38,5 @@
                 <horizontal_fov>1.089</horizontal_fov>
                 <image>
-                    <format>R8G8B8</format>
+                    <format>B8G8R8</format>
                     <width>640</width>
                     <height>480</height>
@@ -50,4 +50,6 @@
                 <plugin name="camera_controller" filename="libgazebo_ros_camera.so">
                     <frame_name>camera_link_optical</frame_name>
+                    <min_depth>0.1</min_depth>
+                    <max_depth>100.0</max_depth>
                 </plugin>
             </plugin>
